Commit message: Restore contributor work, re-apply Gazebo fixes, and cleanup documentation

File: sortabot_description/urdf/sortabot_arms.xacro (robot description, xacro)
@@ -1,6 +1,5 @@
 <?xml version="1.0"?>
 <robot xmlns:xacro="http://www.ros.org/wiki/xacro">
-  <!-- Simple Arm Macro -->
-  <xacro:macro name="simple_arm" params="prefix parent x_offset y_offset color">
+  <xacro:macro name="arm" params="prefix color x_offset y_offset z_offset">
     <link name="${prefix}_arm_base">
       <visual>
@@ -15,11 +14,14 @@
         </geometry>
       </collision>
+      <inertial>
+        <mass value="0.2"/>
+        <inertia ixx="0.001" ixy="0.0" ixz="0.0" iyy="0.001" iyz="0.0" izz="0.001"/>
+      </inertial>
     </link>
     <joint name="${prefix}_base_joint" type="fixed">
-      <parent link="${parent}"/>
+      <parent link="base_link"/>
       <child link="${prefix}_arm_base"/>
-      <origin xyz="${x_offset} ${y_offset} 0.1" rpy="0 0 0"/>
+      <origin xyz="${x_offset} ${y_offset} ${z_offset}" rpy="0 0 0"/>
     </joint>
-    <!-- Link 1 -->
     <link name="${prefix}_link1">
       <visual>
@@ -36,13 +38,17 @@
         </geometry>
       </collision>
+      <inertial>
+        <origin xyz="0 0 0.15" rpy="0 0 0"/>
+        <mass value="0.3"/>
+        <inertia ixx="0.001" ixy="0.0" ixz="0.0" iyy="0.001" iyz="0.0" izz="0.001"/>
+      </inertial>
     </link>
     <joint name="${prefix}_joint1" type="revolute">
       <parent link="${prefix}_arm_base"/>
       <child link="${prefix}_link1"/>
-      <origin xyz="0 0 0.05" rpy="0 0 0"/>
+      <origin xyz="0 0 0.025" rpy="0 0 0"/>
       <axis xyz="0 1 0"/>
-      <limit lower="-1.57" upper="1.57" effort="10.0" velocity="1.0"/>
+      <limit lower="-1.57" upper="1.57" effort="10" velocity="1.0"/>
     </joint>
-    <!-- Hand / End Effector -->
     <link name="${prefix}_hand">
       <visual>
@@ -57,4 +63,8 @@
         </geometry>
       </collision>
+      <inertial>
+        <mass value="0.1"/>
+        <inertia ixx="0.0001" ixy="0.0" ixz="0.0" iyy="0.0001" iyz="0.0" izz="0.0001"/>
+      </inertial>
     </link>
     <!-- Weight Sensor (Virtual Frame) -->
@@ -65,9 +75,11 @@
       <origin xyz="0 0 0.3" rpy="0 0 0"/>
     </joint>
-    <joint name="${prefix}_sensor_joint" type="fixed">
+    <joint name="${prefix}_weight_sensor_joint" type="fixed">
       <parent link="${prefix}_hand"/>
       <child link="${prefix}_weight_sensor"/>
-      <origin xyz="0 0 0" rpy="0 0 0"/>
+      <origin xyz="0 0 0.05" rpy="0 0 0"/>
     </joint>
   </xacro:macro>
+  <xacro:arm prefix="left" color="grey" x_offset="${chassis_length/2 - 0.05}" y_offset="0.12" z_offset="${chassis_height/2 + 0.025}"/>
+  <xacro:arm prefix="right" color="grey" x_offset="${chassis_length/2 - 0.05}" y_offset="-0.12" z_offset="${chassis_height/2 + 0.025}"/>
 </robot>

File: sortabot_description/urdf/sortabot_base.xacro (robot description, xacro)
@@ -1,19 +1,22 @@
 <?xml version="1.0"?>
 <robot xmlns:xacro="http://www.ros.org/wiki/xacro">
-  <!-- Dimensions Placeholder (User to update) -->
-  <xacro:property name="chassis_length" value="0.3"/>
-  <xacro:property name="chassis_width" value="0.2"/>
-  <xacro:property name="chassis_height" value="0.1"/>
-  <xacro:property name="wheel_radius" value="0.05"/>
-  <xacro:property name="wheel_width" value="0.02"/>
+  <xacro:include filename="materials.xacro" />
+  <!-- Constants -->
+  <xacro:property name="chassis_length" value="0.4"/>
+  <xacro:property name="chassis_width" value="0.3"/>
+  <xacro:property name="chassis_height" value="0.15"/>
+  <xacro:property name="wheel_radius" value="0.1"/>
+  <xacro:property name="wheel_width" value="0.04"/>
+  <xacro:property name="wheel_offset" value="0.17"/>
+  <!-- Base footprint (ground projection) -->
   <link name="base_footprint"/>
-  <joint name="base_joint" type="fixed">
+  <joint name="base_footprint_joint" type="fixed">
     <parent link="base_footprint"/>
     <child link="base_link"/>
     <origin xyz="0 0 ${wheel_radius}" rpy="0 0 0"/>
   </joint>
+  <!-- Base Link -->
   <link name="base_link">
     <visual>
-      <origin xyz="0 0 ${chassis_height/2}" rpy="0 0 0"/>
       <geometry>
         <box size="${chassis_length} ${chassis_width} ${chassis_height}"/>
@@ -22,5 +25,4 @@
     </visual>
     <collision>
-      <origin xyz="0 0 ${chassis_height/2}" rpy="0 0 0"/>
       <geometry>
         <box size="${chassis_length} ${chassis_width} ${chassis_height}"/>
@@ -32,5 +34,5 @@
     </inertial>
   </link>
-  <!-- Left Wheel -->
+  <!-- Wheels -->
   <link name="left_wheel">
     <visual>
@@ -45,12 +47,15 @@
       </geometry>
     </collision>
+    <inertial>
+      <mass value="0.1"/>
+      <inertia ixx="0.0001" ixy="0.0" ixz="0.0" iyy="0.0001" iyz="0.0" izz="0.0001"/>
+    </inertial>
   </link>
   <joint name="left_wheel_joint" type="continuous">
     <parent link="base_link"/>
     <child link="left_wheel"/>
-    <origin xyz="0 ${chassis_width/2 + wheel_width/2} 0" rpy="-${pi/2} 0 0"/>
+    <origin xyz="-${chassis_length/4} ${wheel_offset} 0" rpy="-${pi/2} 0 0"/>
     <axis xyz="0 0 1"/>
   </joint>
-  <!-- Right Wheel -->
   <link name="right_wheel">
     <visual>
@@ -65,12 +70,16 @@
       </geometry>
     </collision>
+    <inertial>
+      <mass value="0.1"/>
+      <inertia ixx="0.0001" ixy="0.0" ixz="0.0" iyy="0.0001" iyz="0.0" izz="0.0001"/>
+    </inertial>
   </link>
   <joint name="right_wheel_joint" type="continuous">
     <parent link="base_link"/>
     <child link="right_wheel"/>
-    <origin xyz="0 -${chassis_width/2 + wheel_width/2} 0" rpy="-${pi/2} 0 0"/>
+    <origin xyz="-${chassis_length/4} -${wheel_offset} 0" rpy="-${pi/2} 0 0"/>
     <axis xyz="0 0 1"/>
   </joint>
-  <!-- Caster Wheel -->
+  <!-- Caster -->
   <link name="caster_wheel">
     <visual>
@@ -85,4 +94,8 @@
       </geometry>
     </collision>
+    <inertial>
+      <mass value="0.05"/>
+      <inertia ixx="0.00001" ixy="0.0" ixz="0.0" iyy="0.00001" iyz="0.0" izz="0.00001"/>
+    </inertial>
   </link>
   <joint name="caster_wheel_joint" type="fixed">
@@ -91,3 +104,49 @@
     <origin xyz="${chassis_length/2 - wheel_radius} 0 -${wheel_radius/2}" rpy="0 0 0"/>
   </joint>
+  <!-- Gazebo Physics and Plugins -->
+  <gazebo reference="base_link">
+    <material>Gazebo/Blue</material>
+  </gazebo>
+  <gazebo reference="left_wheel">
+    <material>Gazebo/Black</material>
+    <mu1 value="1.0"/>
+    <mu2 value="1.0"/>
+    <kp value="10000000.0"/>
+    <kd value="1.0"/>
+    <fdir1 value="1 0 0"/>
+  </gazebo>
+  <gazebo reference="right_wheel">
+    <material>Gazebo/Black</material>
+    <mu1 value="1.0"/>
+    <mu2 value="1.0"/>
+    <kp value="10000000.0"/>
+    <kd value="1.0"/>
+    <fdir1 value="1 0 0"/>
+  </gazebo>
+  <gazebo reference="caster_wheel">
+    <material>Gazebo/White</material>
+    <mu1 value="0.001"/>
+    <mu2 value="0.001"/>
+  </gazebo>
+  <gazebo>
+    <plugin
+      filename="gz-sim-diff-drive-system"
+      name="gz::sim::systems::DiffDrive">
+      <left_joint>left_wheel_joint</left_joint>
+      <right_joint>right_wheel_joint</right_joint>
+      <wheel_separation>${chassis_width + wheel_width}</wheel_separation>
+      <wheel_radius>${wheel_radius}</wheel_radius>
+      <odom_publish_frequency>30</odom_publish_frequency>
+      <topic>cmd_vel</topic>
+      <odom_topic>odom</odom_topic>
+      <tf_topic>tf</tf_topic>
+      <frame_id>odom</frame_id>
+      <child_frame_id>base_footprint</child_frame_id>
+    </plugin>
+    <plugin
+      filename="gz-sim-joint-state-publisher-system"
+      name="gz::sim::systems::JointStatePublisher">
+      <topic>joint_states</topic>
+    </plugin>
+  </gazebo>
 </robot>

File: sortabot_description/urdf/sortabot_sensors.xacro (robot description, xacro)
@@ -1,6 +1,4 @@
 <?xml version="1.0"?>
 <robot xmlns:xacro="http://www.ros.org/wiki/xacro">
-  <xacro:macro name="add_sensors" params="parent">
-    <!-- Camera -->
     <link name="camera_link">
       <visual>
@@ -10,11 +8,19 @@
         <material name="black"/>
       </visual>
+      <collision>
+        <geometry>
+          <box size="0.05 0.05 0.05"/>
+        </geometry>
+      </collision>
+      <inertial>
+        <mass value="0.01"/>
+        <inertia ixx="0.00001" ixy="0.0" ixz="0.0" iyy="0.00001" iyz="0.0" izz="0.00001"/>
+      </inertial>
     </link>
     <joint name="camera_joint" type="fixed">
-      <parent link="${parent}"/>
+      <parent link="base_link"/>
       <child link="camera_link"/>
-      <origin xyz="0.14 0 0.12" rpy="0 0 0"/>
+      <origin xyz="${chassis_length/2} 0 ${chassis_height/2}" rpy="0 0 0"/>
     </joint>
-    <!-- LDR / Lidar -->
     <link name="ldr_link">
       <visual>
@@ -24,10 +30,18 @@
         <material name="blue"/>
       </visual>
+      <collision>
+        <geometry>
+          <cylinder radius="0.03" length="0.04"/>
+        </geometry>
+      </collision>
+      <inertial>
+        <mass value="0.01"/>
+        <inertia ixx="0.00001" ixy="0.0" ixz="0.0" iyy="0.00001" iyz="0.0" izz="0.00001"/>
+      </inertial>
     </link>
     <joint name="ldr_joint" type="fixed">
-      <parent link="${parent}"/>
+      <parent link="base_link"/>
       <child link="ldr_link"/>
-      <origin xyz="0 0 0.12" rpy="0 0 0"/>
+      <origin xyz="${chassis_length/2 - 0.05} 0 0.12" rpy="0 0 0"/>
     </joint>
-  </xacro:macro>
 </robot>
