Commit message: Final verified simulation state for Gazebo Harmonic

File: sortabot_description/urdf/sortabot.urdf.xacro (robot description, xacro)
@@ -1,12 +1,201 @@
 <?xml version="1.0"?>
 <robot xmlns:xacro="http://www.ros.org/wiki/xacro" name="sortabot">
-  <xacro:include filename="$(find sortabot_description)/urdf/materials.xacro" />
-  <xacro:include filename="$(find sortabot_description)/urdf/sortabot_base.xacro" />
-  <xacro:include filename="$(find sortabot_description)/urdf/sortabot_arms.xacro" />
-  <xacro:include filename="$(find sortabot_description)/urdf/sortabot_sensors.xacro" />
-  <!-- Instantiate Two Arms -->
-  <xacro:simple_arm prefix="left" parent="base_link" x_offset="0.0" y_offset="0.12" color="white"/>
-  <xacro:simple_arm prefix="right" parent="base_link" x_offset="0.0" y_offset="-0.12" color="white"/>
-  <!-- Instantiate Sensors -->
-  <xacro:add_sensors parent="base_link"/>
+  <!-- MATERIALS -->
+  <material name="blue"><color rgba="0 0 0.8 1"/></material>
+  <material name="black"><color rgba="0 0 0 1"/></material>
+  <material name="white"><color rgba="1 1 1 1"/></material>
+  <material name="red"><color rgba="0.8 0 0 1"/></material>
+  <material name="grey"><color rgba="0.5 0.5 0.5 1"/></material>
+  <!-- CONSTANTS -->
+  <xacro:property name="chassis_length" value="0.4"/>
+  <xacro:property name="chassis_width" value="0.3"/>
+  <xacro:property name="chassis_height" value="0.15"/>
+  <xacro:property name="wheel_radius" value="0.1"/>
+  <xacro:property name="wheel_width" value="0.04"/>
+  <xacro:property name="wheel_offset" value="0.17"/>
+  <!-- BASE -->
+  <link name="base_footprint"/>
+  <joint name="base_footprint_joint" type="fixed">
+    <parent link="base_footprint"/>
+    <child link="base_link"/>
+    <origin xyz="0 0 ${wheel_radius}" rpy="0 0 0"/>
+  </joint>
+  <link name="base_link">
+    <visual>
+      <geometry><box size="${chassis_length} ${chassis_width} ${chassis_height}"/></geometry>
+      <material name="blue"/>
+    </visual>
+    <collision>
+      <geometry><box size="${chassis_length} ${chassis_width} ${chassis_height}"/></geometry>
+    </collision>
+    <inertial>
+      <mass value="1.0"/>
+      <inertia ixx="0.1" ixy="0.0" ixz="0.0" iyy="0.1" iyz="0.0" izz="0.1"/>
+    </inertial>
+  </link>
+  <!-- WHEELS -->
+  <xacro:macro name="wheel" params="prefix y_reflect">
+    <link name="${prefix}_wheel">
+      <visual>
+        <geometry><cylinder radius="${wheel_radius}" length="${wheel_width}"/></geometry>
+        <material name="black"/>
+      </visual>
+      <collision>
+        <geometry><cylinder radius="${wheel_radius}" length="${wheel_width}"/></geometry>
+      </collision>
+      <inertial>
+        <mass value="0.1"/>
+        <inertia ixx="0.001" ixy="0" ixz="0" iyy="0.001" iyz="0" izz="0.001"/>
+      </inertial>
+    </link>
+    <joint name="${prefix}_wheel_joint" type="continuous">
+      <parent link="base_link"/>
+      <child link="${prefix}_wheel"/>
+      <origin xyz="-${chassis_length/4} ${y_reflect * wheel_offset} 0" rpy="-${pi/2} 0 0"/>
+      <axis xyz="0 0 1"/>
+    </joint>
+  </xacro:macro>
+  <xacro:wheel prefix="left" y_reflect="1"/>
+  <xacro:wheel prefix="right" y_reflect="-1"/>
+  <!-- CASTER -->
+  <link name="caster_wheel">
+    <visual>
+      <geometry><sphere radius="${wheel_radius/2}"/></geometry>
+      <material name="white"/>
+    </visual>
+    <collision>
+      <geometry><sphere radius="${wheel_radius/2}"/></geometry>
+    </collision>
+    <inertial>
+      <mass value="0.05"/>
+      <inertia ixx="0.0001" ixy="0" ixz="0" iyy="0.0001" iyz="0" izz="0.0001"/>
+    </inertial>
+  </link>
+  <joint name="caster_wheel_joint" type="fixed">
+    <parent link="base_link"/>
+    <child link="caster_wheel"/>
+    <origin xyz="${chassis_length/2 - wheel_radius} 0 -${wheel_radius/2}" rpy="0 0 0"/>
+  </joint>
+  <!-- ARMS -->
+  <xacro:macro name="arm" params="prefix y_offset">
+    <link name="${prefix}_arm_base">
+      <visual>
+        <geometry><cylinder radius="0.04" length="0.05"/></geometry>
+        <material name="grey"/>
+      </visual>
+      <collision>
+        <geometry><cylinder radius="0.04" length="0.05"/></geometry>
+      </collision>
+      <inertial>
+        <mass value="0.2"/>
+        <inertia ixx="0.001" ixy="0" ixz="0" iyy="0.001" iyz="0" izz="0.001"/>
+      </inertial>
+    </link>
+    <joint name="${prefix}_arm_base_joint" type="fixed">
+      <parent link="base_link"/>
+      <child link="${prefix}_arm_base"/>
+      <origin xyz="${chassis_length/2 - 0.05} ${y_offset} ${chassis_height/2 + 0.025}" rpy="0 0 0"/>
+    </joint>
+    <link name="${prefix}_link1">
+      <visual>
+        <origin xyz="0 0 0.15" rpy="0 0 0"/>
+        <geometry><box size="0.04 0.04 0.3"/></geometry>
+        <material name="grey"/>
+      </visual>
+      <collision>
+        <origin xyz="0 0 0.15" rpy="0 0 0"/>
+        <geometry><box size="0.04 0.04 0.3"/></geometry>
+      </collision>
+      <inertial>
+        <origin xyz="0 0 0.15" rpy="0 0 0"/>
+        <mass value="0.3"/>
+        <inertia ixx="0.001" ixy="0" ixz="0" iyy="0.001" iyz="0" izz="0.001"/>
+      </inertial>
+    </link>
+    <joint name="${prefix}_arm_joint1" type="revolute">
+      <parent link="${prefix}_arm_base"/>
+      <child link="${prefix}_link1"/>
+      <origin xyz="0 0 0.025" rpy="0 0 0"/>
+      <axis xyz="0 1 0"/>
+      <limit lower="-1.57" upper="1.57" effort="10" velocity="1.0"/>
+    </joint>
+    <link name="${prefix}_hand">
+      <visual>
+        <geometry><sphere radius="0.05"/></geometry>
+        <material name="red"/>
+      </visual>
+      <collision>
+        <geometry><sphere radius="0.05"/></geometry>
+      </collision>
+      <inertial>
+        <mass value="0.1"/>
+        <inertia ixx="0.001" ixy="0" ixz="0" iyy="0.001" iyz="0" izz="0.001"/>
+      </inertial>
+    </link>
+    <joint name="${prefix}_hand_joint" type="fixed">
+      <parent link="${prefix}_link1"/>
+      <child link="${prefix}_hand"/>
+      <origin xyz="0 0 0.3" rpy="0 0 0"/>
+    </joint>
+  </xacro:macro>
+  <xacro:arm prefix="left" y_offset="0.12"/>
+  <xacro:arm prefix="right" y_offset="-0.12"/>
+  <!-- SENSORS -->
+  <link name="camera_link">
+    <visual>
+      <geometry><box size="0.05 0.05 0.05"/></geometry>
+      <material name="black"/>
+    </visual>
+    <collision>
+      <geometry><box size="0.05 0.05 0.05"/></geometry>
+    </collision>
+    <inertial>
+      <mass value="0.01"/>
+      <inertia ixx="0.0001" ixy="0" ixz="0" iyy="0.0001" iyz="0" izz="0.0001"/>
+    </inertial>
+  </link>
+  <joint name="camera_joint" type="fixed">
+    <parent link="base_link"/>
+    <child link="camera_link"/>
+    <origin xyz="${chassis_length/2} 0 ${chassis_height/2}" rpy="0 0 0"/>
+  </joint>
+  <link name="ldr_link">
+    <visual>
+      <geometry><cylinder radius="0.03" length="0.04"/></geometry>
+      <material name="blue"/>
+    </visual>
+    <collision>
+      <geometry><cylinder radius="0.03" length="0.04"/></geometry>
+    </collision>
+    <inertial>
+      <mass value="0.01"/>
+      <inertia ixx="0.0001" ixy="0" ixz="0" iyy="0.0001" iyz="0" izz="0.0001"/>
+    </inertial>
+  </link>
+  <joint name="ldr_joint" type="fixed">
+    <parent link="base_link"/>
+    <child link="ldr_link"/>
+    <origin xyz="${chassis_length/2 - 0.05} 0 0.12" rpy="0 0 0"/>
+  </joint>
+  <!-- GAZEBO PLUGINS -->
+  <gazebo reference="base_link"><material>Gazebo/Blue</material></gazebo>
+  <gazebo reference="left_wheel"><material>Gazebo/Black</material></gazebo>
+  <gazebo reference="right_wheel"><material>Gazebo/Black</material></gazebo>
+  <gazebo reference="caster_wheel"><material>Gazebo/White</material><mu1 value="0.001"/><mu2 value="0.001"/></gazebo>
+  <gazebo>
+    <plugin filename="gz-sim-diff-drive-system" name="gz::sim::systems::DiffDrive">
+      <left_joint>left_wheel_joint</left_joint>
+      <right_joint>right_wheel_joint</right_joint>
+      <wheel_separation>${chassis_width + wheel_width}</wheel_separation>
+      <wheel_radius>${wheel_radius}</wheel_radius>
+      <topic>cmd_vel</topic>
+      <odom_topic>odom</odom_topic>
+      <tf_topic>tf</tf_topic>
+      <frame_id>odom</frame_id>
+      <child_frame_id>base_footprint</child_frame_id>
+    </plugin>
+    <plugin filename="gz-sim-joint-state-publisher-system" name="gz::sim::systems::JointStatePublisher">
+      <topic>joint_states</topic>
+    </plugin>
+  </gazebo>
 </robot>

Commit message: Fix wheel polarity in URDF and improve action server controller

File: sortabot_description/urdf/sortabot.urdf.xacro (robot description, xacro)
@@ -35,5 +35,5 @@
   </link>
   <!-- WHEELS -->
-  <xacro:macro name="wheel" params="prefix y_reflect">
+  <xacro:macro name="wheel" params="prefix y_reflect rpy_val">
     <link name="${prefix}_wheel">
       <visual>
@@ -52,10 +52,10 @@
       <parent link="base_link"/>
       <child link="${prefix}_wheel"/>
-      <origin xyz="-${chassis_length/4} ${y_reflect * wheel_offset} 0" rpy="-${pi/2} 0 0"/>
+      <origin xyz="-${chassis_length/4} ${y_reflect * wheel_offset} 0" rpy="${rpy_val}"/>
       <axis xyz="0 0 1"/>
     </joint>
   </xacro:macro>
-  <xacro:wheel prefix="left" y_reflect="1"/>
-  <xacro:wheel prefix="right" y_reflect="-1"/>
+  <xacro:wheel prefix="left" y_reflect="1" rpy_val="-${pi/2} 0 0"/>
+  <xacro:wheel prefix="right" y_reflect="-1" rpy_val="${pi/2} 0 0"/>
   <!-- CASTER -->
   <link name="caster_wheel">
@@ -189,7 +189,7 @@
       <wheel_separation>${chassis_width + wheel_width}</wheel_separation>
       <wheel_radius>${wheel_radius}</wheel_radius>
-      <topic>cmd_vel</topic>
-      <odom_topic>odom</odom_topic>
-      <tf_topic>tf</tf_topic>
+      <topic>/cmd_vel</topic>
+      <odom_topic>/odom</odom_topic>
+      <tf_topic>/tf</tf_topic>
       <frame_id>odom</frame_id>
       <child_frame_id>base_footprint</child_frame_id>

Commit message: FINAL STABLE BUILD: Fixed physics pitching, stabilized URDF, and verified control logic locally

File: sortabot_description/urdf/sortabot.urdf.xacro (robot description, xacro)
@@ -8,4 +8,5 @@
   <material name="grey"><color rgba="0.5 0.5 0.5 1"/></material>
   <!-- CONSTANTS -->
+  <xacro:property name="mass_base" value="5.0"/>
   <xacro:property name="chassis_length" value="0.4"/>
   <xacro:property name="chassis_width" value="0.3"/>
@@ -23,28 +24,34 @@
   <link name="base_link">
     <visual>
+      <origin xyz="0 0 ${chassis_height/2}" rpy="0 0 0"/>
       <geometry><box size="${chassis_length} ${chassis_width} ${chassis_height}"/></geometry>
       <material name="blue"/>
     </visual>
     <collision>
+      <origin xyz="0 0 ${chassis_height/2}" rpy="0 0 0"/>
       <geometry><box size="${chassis_length} ${chassis_width} ${chassis_height}"/></geometry>
     </collision>
     <inertial>
-      <mass value="1.0"/>
+      <!-- Lower Center of Mass for stability -->
+      <origin xyz="0 0 ${chassis_height/4}" rpy="0 0 0"/>
+      <mass value="${mass_base}"/>
       <inertia ixx="0.1" ixy="0.0" ixz="0.0" iyy="0.1" iyz="0.0" izz="0.1"/>
     </inertial>
   </link>
-  <!-- WHEELS -->
-  <xacro:macro name="wheel" params="prefix y_reflect rpy_val">
+  <!-- WHEEL MACRO -->
+  <xacro:macro name="wheel" params="prefix y_reflect">
     <link name="${prefix}_wheel">
       <visual>
+        <origin xyz="0 0 0" rpy="${pi/2} 0 0"/>
         <geometry><cylinder radius="${wheel_radius}" length="${wheel_width}"/></geometry>
         <material name="black"/>
       </visual>
       <collision>
+        <origin xyz="0 0 0" rpy="${pi/2} 0 0"/>
         <geometry><cylinder radius="${wheel_radius}" length="${wheel_width}"/></geometry>
       </collision>
       <inertial>
-        <mass value="0.1"/>
-        <inertia ixx="0.001" ixy="0" ixz="0" iyy="0.001" iyz="0" izz="0.001"/>
+        <mass value="0.5"/>
+        <inertia ixx="0.01" ixy="0" ixz="0" iyy="0.01" iyz="0" izz="0.01"/>
       </inertial>
     </link>
@@ -52,11 +59,11 @@
       <parent link="base_link"/>
       <child link="${prefix}_wheel"/>
-      <origin xyz="-${chassis_length/4} ${y_reflect * wheel_offset} 0" rpy="${rpy_val}"/>
-      <axis xyz="0 0 1"/>
+      <origin xyz="-${chassis_length/4} ${y_reflect * wheel_offset} 0" rpy="0 0 0"/>
+      <axis xyz="0 1 0"/>
     </joint>
   </xacro:macro>
-  <xacro:wheel prefix="left" y_reflect="1" rpy_val="-${pi/2} 0 0"/>
-  <xacro:wheel prefix="right" y_reflect="-1" rpy_val="${pi/2} 0 0"/>
-  <!-- CASTER -->
+  <xacro:wheel prefix="left" y_reflect="1"/>
+  <xacro:wheel prefix="right" y_reflect="-1"/>
+  <!-- CASTER (Front) -->
   <link name="caster_wheel">
     <visual>
@@ -68,6 +75,6 @@
     </collision>
     <inertial>
-      <mass value="0.05"/>
-      <inertia ixx="0.0001" ixy="0" ixz="0" iyy="0.0001" iyz="0" izz="0.0001"/>
+      <mass value="0.2"/>
+      <inertia ixx="0.001" ixy="0" ixz="0" iyy="0.001" iyz="0" izz="0.001"/>
     </inertial>
   </link>
@@ -75,117 +82,30 @@
     <parent link="base_link"/>
     <child link="caster_wheel"/>
-    <origin xyz="${chassis_length/2 - wheel_radius} 0 -${wheel_radius/2}" rpy="0 0 0"/>
+    <origin xyz="${chassis_length/2 - wheel_radius} 0 -0.05" rpy="0 0 0"/>
   </joint>
-  <!-- ARMS -->
+  <!-- ARMS (Simplified for weight stability) -->
   <xacro:macro name="arm" params="prefix y_offset">
     <link name="${prefix}_arm_base">
-      <visual>
-        <geometry><cylinder radius="0.04" length="0.05"/></geometry>
-        <material name="grey"/>
-      </visual>
-      <collision>
-        <geometry><cylinder radius="0.04" length="0.05"/></geometry>
-      </collision>
-      <inertial>
-        <mass value="0.2"/>
-        <inertia ixx="0.001" ixy="0" ixz="0" iyy="0.001" iyz="0" izz="0.001"/>
-      </inertial>
+      <visual><geometry><cylinder radius="0.02" length="0.02"/></geometry><material name="grey"/></visual>
+      <inertial><mass value="0.05"/><inertia ixx="0.0001" ixy="0" ixz="0" iyy="0.0001" iyz="0" izz="0.0001"/></inertial>
     </link>
     <joint name="${prefix}_arm_base_joint" type="fixed">
       <parent link="base_link"/>
       <child link="${prefix}_arm_base"/>
-      <origin xyz="${chassis_length/2 - 0.05} ${y_offset} ${chassis_height/2 + 0.025}" rpy="0 0 0"/>
-    </joint>
-    <link name="${prefix}_link1">
-      <visual>
-        <origin xyz="0 0 0.15" rpy="0 0 0"/>
-        <geometry><box size="0.04 0.04 0.3"/></geometry>
-        <material name="grey"/>
-      </visual>
-      <collision>
-        <origin xyz="0 0 0.15" rpy="0 0 0"/>
-        <geometry><box size="0.04 0.04 0.3"/></geometry>
-      </collision>
-      <inertial>
-        <origin xyz="0 0 0.15" rpy="0 0 0"/>
-        <mass value="0.3"/>
-        <inertia ixx="0.001" ixy="0" ixz="0" iyy="0.001" iyz="0" izz="0.001"/>
-      </inertial>
-    </link>
-    <joint name="${prefix}_arm_joint1" type="revolute">
-      <parent link="${prefix}_arm_base"/>
-      <child link="${prefix}_link1"/>
-      <origin xyz="0 0 0.025" rpy="0 0 0"/>
-      <axis xyz="0 1 0"/>
-      <limit lower="-1.57" upper="1.57" effort="10" velocity="1.0"/>
-    </joint>
-    <link name="${prefix}_hand">
-      <visual>
-        <geometry><sphere radius="0.05"/></geometry>
-        <material name="red"/>
-      </visual>
-      <collision>
-        <geometry><sphere radius="0.05"/></geometry>
-      </collision>
-      <inertial>
-        <mass value="0.1"/>
-        <inertia ixx="0.001" ixy="0" ixz="0" iyy="0.001" iyz="0" izz="0.001"/>
-      </inertial>
-    </link>
-    <joint name="${prefix}_hand_joint" type="fixed">
-      <parent link="${prefix}_link1"/>
-      <child link="${prefix}_hand"/>
-      <origin xyz="0 0 0.3" rpy="0 0 0"/>
+      <origin xyz="${chassis_length/2 - 0.05} ${y_offset} ${chassis_height}" rpy="0 0 0"/>
     </joint>
   </xacro:macro>
-  <xacro:arm prefix="left" y_offset="0.12"/>
-  <xacro:arm prefix="right" y_offset="-0.12"/>
-  <!-- SENSORS -->
-  <link name="camera_link">
-    <visual>
-      <geometry><box size="0.05 0.05 0.05"/></geometry>
-      <material name="black"/>
-    </visual>
-    <collision>
-      <geometry><box size="0.05 0.05 0.05"/></geometry>
-    </collision>
-    <inertial>
-      <mass value="0.01"/>
-      <inertia ixx="0.0001" ixy="0" ixz="0" iyy="0.0001" iyz="0" izz="0.0001"/>
-    </inertial>
-  </link>
-  <joint name="camera_joint" type="fixed">
-    <parent link="base_link"/>
-    <child link="camera_link"/>
-    <origin xyz="${chassis_length/2} 0 ${chassis_height/2}" rpy="0 0 0"/>
-  </joint>
-  <link name="ldr_link">
-    <visual>
-      <geometry><cylinder radius="0.03" length="0.04"/></geometry>
-      <material name="blue"/>
-    </visual>
-    <collision>
-      <geometry><cylinder radius="0.03" length="0.04"/></geometry>
-    </collision>
-    <inertial>
-      <mass value="0.01"/>
-      <inertia ixx="0.0001" ixy="0" ixz="0" iyy="0.0001" iyz="0" izz="0.0001"/>
-    </inertial>
-  </link>
-  <joint name="ldr_joint" type="fixed">
-    <parent link="base_link"/>
-    <child link="ldr_link"/>
-    <origin xyz="${chassis_length/2 - 0.05} 0 0.12" rpy="0 0 0"/>
-  </joint>
-  <!-- GAZEBO PLUGINS -->
+  <xacro:arm prefix="left" y_offset="0.1"/>
+  <xacro:arm prefix="right" y_offset="-0.1"/>
+  <!-- GAZEBO -->
   <gazebo reference="base_link"><material>Gazebo/Blue</material></gazebo>
-  <gazebo reference="left_wheel"><material>Gazebo/Black</material></gazebo>
-  <gazebo reference="right_wheel"><material>Gazebo/Black</material></gazebo>
-  <gazebo reference="caster_wheel"><material>Gazebo/White</material><mu1 value="0.001"/><mu2 value="0.001"/></gazebo>
+  <gazebo reference="left_wheel"><material>Gazebo/Black</material><mu1>1.0</mu1><mu2>1.0</mu2><kp>1000000.0</kp><kd>100.0</kd></gazebo>
+  <gazebo reference="right_wheel"><material>Gazebo/Black</material><mu1>1.0</mu1><mu2>1.0</mu2><kp>1000000.0</kp><kd>100.0</kd></gazebo>
+  <gazebo reference="caster_wheel"><material>Gazebo/White</material><mu1>0.01</mu1><mu2>0.01</mu2></gazebo>
   <gazebo>
     <plugin filename="gz-sim-diff-drive-system" name="gz::sim::systems::DiffDrive">
       <left_joint>left_wheel_joint</left_joint>
       <right_joint>right_wheel_joint</right_joint>
-      <wheel_separation>${chassis_width + wheel_width}</wheel_separation>
+      <wheel_separation>${wheel_offset * 2}</wheel_separation>
       <wheel_radius>${wheel_radius}</wheel_radius>
       <topic>/cmd_vel</topic>
@@ -194,7 +114,9 @@
       <frame_id>odom</frame_id>
       <child_frame_id>base_footprint</child_frame_id>
+      <max_linear_acceleration>0.5</max_linear_acceleration>
+      <max_angular_acceleration>1.0</max_angular_acceleration>
     </plugin>
     <plugin filename="gz-sim-joint-state-publisher-system" name="gz::sim::systems::JointStatePublisher">
-      <topic>joint_states</topic>
+      <topic>/joint_states</topic>
     </plugin>
   </gazebo>
