Commit message: Updated files for spawning dumbbells

File: final_dumbbell.urdf (robot description, URDF)
Before this commit: robot dumbbell_pure, 4 links, 3 joints
Links:
- removed link handle
- removed link left_w
- removed link right_w
- link base_link: mass None -> 5.0; geometry collision cylinder length=0.2 radius=0.02; collision sphere radius=0.06
Joints:
- removed joint joint_left
- removed joint joint_right
- removed joint root_joint
